File: hardware/xmas_v2/xmas_v2.sch (EAGLE design)
At the start: 0 parts

Commit message: Added all parts
Parts:
- added BAT1: 3V, SparkFun-Electromechanical:BATTERY20PTH
- added BLU0, BLU12, BLU15, BLU3, BLU6, BLU9: (no value), SparkFun-LED:LED5MM-KIT
- added C1: .1uf, SparkFun-Capacitors:CAP0805
- added GRN11, GRN14, GRN17, GRN2, GRN5, GRN8, RED1, RED10, RED13, RED16, RED4, RED7: (no value), adafruit:LEDCHIPLED_0805
- added JP1, JP2: (no value), SparkFun-Connectors:M01NOSILK-KIT
- added R1, R2, R3, R4, R5: 100, SparkFun-Passives:RESISTOR0805-RES
- added R6: 10K, SparkFun-Passives:RESISTOR0805-RES
- added S1: SWITCH-MOMENTARY-2SMD-4, SparkFun-Electromechanical:SWITCH-MOMENTARY-2SMD-4
- added U$1: ATTINY13SOIC, SparkFun-DigitalIC:ATTINY13SOIC
Connections:
- new net PB0: BLU9.A, GRN11.A, GRN8.A, RED10.A
- new net PB1: BLU12.A, BLU15.A, GRN14.A, RED13.A
- new net PB2: GRN17.A, RED16.A
- new net PB3: BLU0.A, BLU3.A, GRN2.A, RED1.A
- new net PB4: BLU6.A, GRN5.A, RED4.A, RED7.A
