File: hardware/xmas_v2/xmas_v2.brd (EAGLE design)
At the start: 109.5 x 100 mm, 30 parts

Commit message: Finished routing
Parts:
- BLU0: value (none) -> 0
- BLU12: value (none) -> 12
- BLU15: value (none) -> 15
- BLU3: value (none) -> 3
- BLU6: value (none) -> 6
- BLU9: value (none) -> 9
- GRN11: value (none) -> 11
- GRN14: value (none) -> 14
- GRN17: value (none) -> 17
- GRN2: value (none) -> 2
- GRN5: value (none) -> 5
- GRN8: value (none) -> 8
- RED1: value (none) -> 1
- RED10: value (none) -> 10
- RED13: value (none) -> 13
- RED16: value (none) -> 16
- RED4: value (none) -> 4
- RED7: value (none) -> 7
- moved C1 27.9 mm to (27.0, 25.0), turned to 0 degrees
- moved R2 7.25 mm to (27.8, 16.8)
- moved R6 4.19 mm to (29.2, 22.0), turned to 180 degrees
- moved R1 1.60 mm to (29.2, 20.0), turned to 0 degrees
- moved R3 1.60 mm to (14.8, 22.0), turned to 180 degrees
- moved R4 1.25 mm to (14.8, 20.0), turned to 180 degrees
- moved R5 0.35 mm to (16.2, 16.8), turned to 270 degrees
- moved JP1 0.25 mm to (26.8, 45.0)
- moved JP2 0.25 mm to (17.2, 45.0)
- turned GRN17 to 255 degrees
- turned GRN8 to 255 degrees
- turned RED1 to 285 degrees
- turned RED16 to 165 degrees
- turned RED7 to 165 degrees
Connections:
- net GND: no longer JP1.1, JP2.1
Routing:
- net PB4: track 0.00 -> 75.5 mm, vias 0 -> 4
- net PB3: track 0.00 -> 69.7 mm, vias 0 -> 5
- net PB2: track 0.00 -> 69.4 mm, vias 0 -> 6
- net PB1: track 0.00 -> 55.8 mm, vias 0 -> 5
- net PB0: track 0.00 -> 52.8 mm, vias 0 -> 3
- net N$1: track 0.00 -> 51.7 mm, vias 0 -> 3
- net N$4: track 0.00 -> 38.2 mm, vias 0 -> 3
- net N$3: track 0.00 -> 37.3 mm, vias 0 -> 2
- net N$2: track 0.00 -> 33.1 mm
- net N$5: track 0.00 -> 28.3 mm, vias 0 -> 2
- net VCC: track 0.00 -> 21.9 mm
- net N$10: track 0.00 -> 11.9 mm
- added copper zone on layer 1, net GND
- added copper zone on layer 16, net GND
Other:
- board size 109.5 x 100 mm -> 109.5 x 87.7 mm

Commit message: Minor routing changes
Routing:
- net N$5: track 28.3 -> 29.3 mm
- net PB4: track 75.5 -> 76.5 mm
- net N$10: track 11.9 -> 12.8 mm
- net PB0: track 52.8 -> 53.3 mm
Other:
- board size 109.5 x 87.7 mm -> 43.3 x 50 mm
- board text added: "2015"
- board text added: "3V CR2032"
- board text added: "Merry Christmas from Blake"
- board text added: "xmas_v2"
